Commit message: V1.6

File: src/quadruped_ros2_control-humble/descriptions/unitree/go1_description/xacro/const.xacro (robot description, xacro)
@@ -54,13 +54,13 @@
 	<xacro:property name="hip_position_min" value="-0.863"/>
 	<xacro:property name="hip_velocity_max" value="30.1"/>
-	<xacro:property name="hip_torque_max" value="53.7"/>
+	<xacro:property name="hip_torque_max" value="1.0"/>
 	<xacro:property name="thigh_position_max" value="4.501"/>
-	<xacro:property name="thigh_position_min" value="-0.686"/>
+	<xacro:property name="thigh_position_min" value="-2.1"/>
 	<xacro:property name="thigh_velocity_max" value="30.1"/>
-	<xacro:property name="thigh_torque_max" value="53.7"/>
+	<xacro:property name="thigh_torque_max" value="1.0"/>
 	<xacro:property name="calf_position_max" value="-0.888"/>
 	<xacro:property name="calf_position_min" value="-2.818"/>
 	<xacro:property name="calf_velocity_max" value="20.06"/>
-	<xacro:property name="calf_torque_max" value="65.55"/>
+	<xacro:property name="calf_torque_max" value="1.0"/>
 	<!-- dynamics inertial value        total 26.0382kg -->
 	<!-- trunk -->
