Commit message: 5

File: src/quadruped_ros2_control-humble/descriptions/sysu219/sysu219_description/urdf/robot.urdf (robot description, URDF)
Before this commit: robot sysu219, 46 links, 45 joints
Links:
- removed link camera_chin
- removed link camera_face
- removed link camera_laserscan_link_left
- removed link camera_laserscan_link_right
- removed link camera_left
- removed link camera_optical_chin
- removed link camera_optical_face
- removed link camera_optical_left
- removed link camera_optical_rearDown
- removed link camera_optical_right
- removed link camera_rearDown
- removed link camera_right
- removed link ultraSound_face
- removed link ultraSound_left
- removed link ultraSound_right
- link FL_calf: mass 0.135862 -> 0.384261; geometry collision box size=0.2835 0.016 0.016; visual mesh filename=file:///home/yzz/219_ws/install/sysu219_description/share/s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 scale=0.001 0.001 0.001
- link FL_calf_rotor: mass 0.089 -> 0.092882; geometry visual cylinder length=0.05 radius=0.056
- link FL_foot: mass 0.06 -> 0.062617
- link FL_hip: mass 0.591 -> 1.619802; geometry collision cylinder length=0.2075 radius=0.0645; visual mesh filename=file:///home/yzz/219_ws/install/sysu219_description/share/s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 scale=0.001 0.001 0.001
- link FL_hip_rotor: mass 0.089 -> 0.092882; geometry visual cylinder length=0.050 radius=0.056
- link FL_thigh: mass 0.92 -> 2.056974; geometry collision box size=0.2835 0.0245 0.034; visual mesh filename=file:///home/yzz/219_ws/install/sysu219_description/share/s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 scale=0.001 0.001 0.001
- link FL_thigh_rotor: mass 0.089 -> 0.092882; geometry visual cylinder length=0.05 radius=0.056
- link FR_calf: mass 0.135862 -> 0.384261; geometry collision box size=0.2835 0.016 0.016; visual mesh filename=file:///home/yzz/219_ws/install/sysu219_description/share/s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 scale=0.001 0.001 0.001
- link FR_calf_rotor: mass 0.089 -> 0.092882; geometry visual cylinder length=0.05 radius=0.056
- link FR_foot: mass 0.06 -> 0.062617
- link FR_hip: mass 0.591 -> 1.619802; geometry collision cylinder length=0.2075 radius=0.0645; visual mesh filename=file:///home/yzz/219_ws/install/sysu219_description/share/s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 scale=0.001 0.001 0.001
- link FR_hip_rotor: mass 0.089 -> 0.092882; geometry visual cylinder length=0.050 radius=0.056
- link FR_thigh: mass 0.92 -> 2.056974; geometry collision box size=0.2835 0.0245 0.034; visual mesh filename=file:///home/yzz/219_ws/install/sysu219_description/share/s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 scale=0.001 0.001 0.001
- link FR_thigh_rotor: mass 0.089 -> 0.092882; geometry visual cylinder length=0.05 radius=0.056
- link RL_calf: mass 0.135862 -> 0.384261; geometry collision box size=0.2835 0.016 0.016; visual mesh filename=file:///home/yzz/219_ws/install/sysu219_description/share/s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 scale=0.001 0.001 0.001
- link RL_calf_rotor: mass 0.089 -> 0.092882; geometry visual cylinder length=0.05 radius=0.056
- link RL_foot: mass 0.06 -> 0.062617
- link RL_hip: mass 0.591 -> 1.619802; geometry collision cylinder length=0.2075 radius=0.0645; visual mesh filename=file:///home/yzz/219_ws/install/sysu219_description/share/s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 scale=0.001 0.001 0.001
- link RL_hip_rotor: mass 0.089 -> 0.092882; geometry visual cylinder length=0.050 radius=0.056
- link RL_thigh: mass 0.92 -> 2.056974; geometry collision box size=0.2835 0.0245 0.034; visual mesh filename=file:///home/yzz/219_ws/install/sysu219_description/share/s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 scale=0.001 0.001 0.001
- link RL_thigh_rotor: mass 0.089 -> 0.092882; geometry visual cylinder length=0.05 radius=0.056
- link RR_calf: mass 0.135862 -> 0.384261; geometry collision box size=0.2835 0.016 0.016; visual mesh filename=file:///home/yzz/219_ws/install/sysu219_description/share/s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 scale=0.001 0.001 0.001
- link RR_calf_rotor: mass 0.089 -> 0.092882; geometry visual cylinder length=0.05 radius=0.056
- link RR_foot: mass 0.06 -> 0.062617
- link RR_hip: mass 0.591 -> 1.619802; geometry collision cylinder length=0.2075 radius=0.0645; visual mesh filename=file:///home/yzz/219_ws/install/sysu219_description/share/s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 scale=0.001 0.001 0.001
- link RR_hip_rotor: mass 0.089 -> 0.092882; geometry visual cylinder length=0.050 radius=0.056
- link RR_thigh: mass 0.92 -> 2.056974; geometry collision box size=0.2835 0.0245 0.034; visual mesh filename=file:///home/yzz/219_ws/install/sysu219_description/share/s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 scale=0.001 0.001 0.001
- link RR_thigh_rotor: mass 0.089 -> 0.092882; geometry visual cylinder length=0.05 radius=0.056
- link trunk: mass 5.204 -> 22.8908; geometry collision box size=0.8575 0.32 0.23; visual mesh filename=file:///home/yzz/219_ws/install/sysu219_description/share/s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 scale=0.001 0.001 0.001
Joints:
- removed joint camera_joint_chin
- removed joint camera_joint_face
- removed joint camera_joint_left
- removed joint camera_joint_rearDown
- removed joint camera_joint_right
- removed joint camera_laserscan_joint_left
- removed joint camera_laserscan_joint_right
- removed joint camera_optical_joint_chin
- removed joint camera_optical_joint_face
- removed joint camera_optical_joint_left
- removed joint camera_optical_joint_rearDown
- removed joint camera_optical_joint_right
- removed joint ultraSound_joint_face
- removed joint ultraSound_joint_left
- removed joint ultraSound_joint_right
- joint FL_calf_joint: limit lower=-2.818 upper=-0.888 effort=35.55 velocity=20.06 -> lower=-2.818 upper=-0.888 effort=100.0 velocity=20.06; origin xyz=0 0 -0.213 rpy=0 0 0 -> xyz=0 0 -0.2835 rpy=0 0 0
- joint FL_calf_rotor_joint: origin xyz=0.0 -0.03235 0 rpy=0 0 0 -> xyz=0.0 -0.06055 0 rpy=0 0 0
- joint FL_foot_fixed: origin xyz=0 0 -0.213 rpy=0 0 0 -> xyz=0 0 -0.2835 rpy=0 0 0
- joint FL_hip_joint: limit lower=-0.863 upper=0.863 effort=23.7 velocity=30.1 -> lower=-0.863 upper=0.863 effort=100.0 velocity=30.1; origin xyz=0.1881 0.04675 0 rpy=0 0 0 -> xyz=0.34525 0.094 0 rpy=0 0 0
- joint FL_hip_rotor_joint: origin xyz=0.11215 0.04675 0 rpy=0 0 0 -> xyz=0.21525 0.094 0 rpy=0 0 0
- joint FL_thigh_joint: limit lower=-0.686 upper=4.501 effort=23.7 velocity=30.1 -> lower=-2.1 upper=4.501 effort=100.0 velocity=30.1; origin xyz=0 0.08 0 rpy=0 0 0 -> xyz=0 0.1243 0 rpy=0 0 0
- joint FL_thigh_rotor_joint: origin xyz=0.0 -0.00015 0 rpy=0 0 0 -> xyz=0.0 -0.03675 0 rpy=0 0 0
- joint FR_calf_joint: limit lower=-2.818 upper=-0.888 effort=35.55 velocity=20.06 -> lower=-2.818 upper=-0.888 effort=100.0 velocity=20.06; origin xyz=0 0 -0.213 rpy=0 0 0 -> xyz=0 0 -0.2835 rpy=0 0 0
- joint FR_calf_rotor_joint: origin xyz=0.0 0.03235 0 rpy=0 0 0 -> xyz=0.0 0.06055 0 rpy=0 0 0
- joint FR_foot_fixed: origin xyz=0 0 -0.213 rpy=0 0 0 -> xyz=0 0 -0.2835 rpy=0 0 0
- joint FR_hip_joint: limit lower=-0.863 upper=0.863 effort=23.7 velocity=30.1 -> lower=-0.863 upper=0.863 effort=100.0 velocity=30.1; origin xyz=0.1881 -0.04675 0 rpy=0 0 0 -> xyz=0.34525 -0.094 0 rpy=0 0 0
- joint FR_hip_rotor_joint: origin xyz=0.11215 -0.04675 0 rpy=0 0 0 -> xyz=0.21525 -0.094 0 rpy=0 0 0
- joint FR_thigh_joint: limit lower=-0.686 upper=4.501 effort=23.7 velocity=30.1 -> lower=-2.1 upper=4.501 effort=100.0 velocity=30.1; origin xyz=0 -0.08 0 rpy=0 0 0 -> xyz=0 -0.1243 0 rpy=0 0 0
- joint FR_thigh_rotor_joint: origin xyz=0.0 0.00015 0 rpy=0 0 0 -> xyz=0.0 0.03675 0 rpy=0 0 0
- joint RL_calf_joint: limit lower=-2.818 upper=-0.888 effort=35.55 velocity=20.06 -> lower=-2.818 upper=-0.888 effort=100.0 velocity=20.06; origin xyz=0 0 -0.213 rpy=0 0 0 -> xyz=0 0 -0.2835 rpy=0 0 0
- joint RL_calf_rotor_joint: origin xyz=0.0 -0.03235 0 rpy=0 0 0 -> xyz=0.0 -0.06055 0 rpy=0 0 0
- joint RL_foot_fixed: origin xyz=0 0 -0.213 rpy=0 0 0 -> xyz=0 0 -0.2835 rpy=0 0 0
- joint RL_hip_joint: limit lower=-0.863 upper=0.863 effort=23.7 velocity=30.1 -> lower=-0.863 upper=0.863 effort=100.0 velocity=30.1; origin xyz=-0.1881 0.04675 0 rpy=0 0 0 -> xyz=-0.34525 0.094 0 rpy=0 0 0
- joint RL_hip_rotor_joint: origin xyz=-0.11215 0.04675 0 rpy=0 0 0 -> xyz=-0.21525 0.094 0 rpy=0 0 0
- joint RL_thigh_joint: limit lower=-0.686 upper=4.501 effort=23.7 velocity=30.1 -> lower=-2.1 upper=4.501 effort=100.0 velocity=30.1; origin xyz=0 0.08 0 rpy=0 0 0 -> xyz=0 0.1243 0 rpy=0 0 0
- joint RL_thigh_rotor_joint: origin xyz=0.0 -0.00015 0 rpy=0 0 0 -> xyz=0.0 -0.03675 0 rpy=0 0 0
- joint RR_calf_joint: limit lower=-2.818 upper=-0.888 effort=35.55 velocity=20.06 -> lower=-2.818 upper=-0.888 effort=100.0 velocity=20.06; origin xyz=0 0 -0.213 rpy=0 0 0 -> xyz=0 0 -0.2835 rpy=0 0 0
- joint RR_calf_rotor_joint: origin xyz=0.0 0.03235 0 rpy=0 0 0 -> xyz=0.0 0.06055 0 rpy=0 0 0
- joint RR_foot_fixed: origin xyz=0 0 -0.213 rpy=0 0 0 -> xyz=0 0 -0.2835 rpy=0 0 0
- joint RR_hip_joint: limit lower=-0.863 upper=0.863 effort=23.7 velocity=30.1 -> lower=-0.863 upper=0.863 effort=100.0 velocity=30.1; origin xyz=-0.1881 -0.04675 0 rpy=0 0 0 -> xyz=-0.34525 -0.094 0 rpy=0 0 0
- joint RR_hip_rotor_joint: origin xyz=-0.11215 -0.04675 0 rpy=0 0 0 -> xyz=-0.21525 -0.094 0 rpy=0 0 0
- joint RR_thigh_joint: limit lower=-0.686 upper=4.501 effort=23.7 velocity=30.1 -> lower=-2.1 upper=4.501 effort=100.0 velocity=30.1; origin xyz=0 -0.08 0 rpy=0 0 0 -> xyz=0 -0.1243 0 rpy=0 0 0
- joint RR_thigh_rotor_joint: origin xyz=0.0 0.00015 0 rpy=0 0 0 -> xyz=0.0 0.03675 0 rpy=0 0 0

File: src/quadruped_ros2_control-humble/descriptions/sysu219/sysu219_description/xacro/const.xacro (robot description, xacro)
@@ -63,80 +63,80 @@
 	<xacro:property name="calf_velocity_max" value="20.06"/>
 	<xacro:property name="calf_torque_max" value="100.0"/>
-	<!-- dynamics inertial value        total 26.0382kg -->
+	<!-- dynamics inertial value        total 40.5kg -->
 	<!-- trunk -->
-	<xacro:property name="trunk_mass" value="10.473"/>
+	<xacro:property name="trunk_mass" value="22.8908"/>
 	<xacro:property name="trunk_com_x" value="-0.0083979"/>
 	<xacro:property name="trunk_com_y" value="0.00014075"/>
 	<xacro:property name="trunk_com_z" value="-0.003899"/>
-	<xacro:property name="trunk_ixx" value="0.069588"/>
-	<xacro:property name="trunk_ixy" value="0.000079993"/>
-	<xacro:property name="trunk_ixz" value="-0.000069927"/>
-	<xacro:property name="trunk_iyy" value="0.14986"/>
-	<xacro:property name="trunk_iyz" value="-0.0000043683"/>
-	<xacro:property name="trunk_izz" value="0.17323"/>
+	<xacro:property name="trunk_ixx" value="0.152098"/>
+	<xacro:property name="trunk_ixy" value="0.000174840"/>
+	<xacro:property name="trunk_ixz" value="-0.000152839"/>
+	<xacro:property name="trunk_iyy" value="0.327548"/>
+	<xacro:property name="trunk_iyz" value="-0.000009548"/>
+	<xacro:property name="trunk_izz" value="0.378628"/>
 	<!-- hip (left front) -->
-	<xacro:property name="hip_mass" value="1.5521"/>
+	<xacro:property name="hip_mass" value="1.619802"/>
 	<xacro:property name="hip_com_x" value="-0.0081895"/>
 	<xacro:property name="hip_com_y" value="-0.0059007"/>
 	<xacro:property name="hip_com_z" value="0.000064549"/>
-	<xacro:property name="hip_ixx" value="0.0013197"/>
-	<xacro:property name="hip_ixy" value="-0.000014496"/>
-	<xacro:property name="hip_ixz" value="0.00000019362"/>
-	<xacro:property name="hip_iyy" value="0.00276"/>
-	<xacro:property name="hip_iyz" value="-0.000011682"/>
-	<xacro:property name="hip_izz" value="0.0017432"/>
-	<xacro:property name="hip_rotor_mass" value="0.089"/>
+	<xacro:property name="hip_ixx" value="0.001377265"/>
+	<xacro:property name="hip_ixy" value="-0.0000151283"/>
+	<xacro:property name="hip_ixz" value="0.000000202066"/>
+	<xacro:property name="hip_iyy" value="0.002880390"/>
+	<xacro:property name="hip_iyz" value="-0.0000121916"/>
+	<xacro:property name="hip_izz" value="0.001819237"/>
+	<xacro:property name="hip_rotor_mass" value="0.092882"/>
 	<xacro:property name="hip_rotor_com_x" value="0.0"/>
 	<xacro:property name="hip_rotor_com_y" value="0.0"/>
 	<xacro:property name="hip_rotor_com_z" value="0.0"/>
-	<xacro:property name="hip_rotor_ixx" value="0.000111842"/>
+	<xacro:property name="hip_rotor_ixx" value="0.000116720"/>
 	<xacro:property name="hip_rotor_ixy" value="0.0"/>
 	<xacro:property name="hip_rotor_ixz" value="0.0"/>
-	<xacro:property name="hip_rotor_iyy" value="0.000059647"/>
+	<xacro:property name="hip_rotor_iyy" value="0.000062249"/>
 	<xacro:property name="hip_rotor_iyz" value="0.0"/>
-	<xacro:property name="hip_rotor_izz" value="0.000059647"/>
+	<xacro:property name="hip_rotor_izz" value="0.000062249"/>
 	<!-- thigh -->
-	<xacro:property name="thigh_mass" value="1.971"/>
+	<xacro:property name="thigh_mass" value="2.056974"/>
 	<xacro:property name="thigh_com_x" value="0.022476"/>
 	<xacro:property name="thigh_com_y" value="-0.020306"/>
 	<xacro:property name="thigh_com_z" value="-0.053334"/>
-	<xacro:property name="thigh_ixx" value="0.0072651"/>
-	<xacro:property name="thigh_ixy" value="0.000040929"/>
-	<xacro:property name="thigh_ixz" value="0.0027107"/>
-	<xacro:property name="thigh_iyy" value="0.010008"/>
-	<xacro:property name="thigh_iyz" value="-0.000098371"/>
-	<xacro:property name="thigh_izz" value="0.0030303"/>
-	<xacro:property name="thigh_rotor_mass" value="0.089"/>
+	<xacro:property name="thigh_ixx" value="0.007582000"/>
+	<xacro:property name="thigh_ixy" value="0.0000427143"/>
+	<xacro:property name="thigh_ixz" value="0.002828939"/>
+	<xacro:property name="thigh_iyy" value="0.010444544"/>
+	<xacro:property name="thigh_iyz" value="-0.000102662"/>
+	<xacro:property name="thigh_izz" value="0.003162480"/>
+	<xacro:property name="thigh_rotor_mass" value="0.092882"/>
 	<xacro:property name="thigh_rotor_com_x" value="0.0"/>
 	<xacro:property name="thigh_rotor_com_y" value="0.0"/>
 	<xacro:property name="thigh_rotor_com_z" value="0.0"/>
-	<xacro:property name="thigh_rotor_ixx" value="0.000059647"/>
+	<xacro:property name="thigh_rotor_ixx" value="0.000062249"/>
 	<xacro:property name="thigh_rotor_ixy" value="0.0"/>
 	<xacro:property name="thigh_rotor_ixz" value="0.0"/>
-	<xacro:property name="thigh_rotor_iyy" value="0.000111842"/>
+	<xacro:property name="thigh_rotor_iyy" value="0.000116720"/>
 	<xacro:property name="thigh_rotor_iyz" value="0.0"/>
-	<xacro:property name="thigh_rotor_izz" value="0.000059647"/>
+	<xacro:property name="thigh_rotor_izz" value="0.000062249"/>
 	<!-- calf -->
-	<xacro:property name="calf_mass" value="0.3682"/>
+	<xacro:property name="calf_mass" value="0.384261"/>
 	<xacro:property name="calf_com_x" value="0.011177"/>
 	<xacro:property name="calf_com_y" value="0.00002257"/>
 	<xacro:property name="calf_com_z" value="-0.15282"/>
-	<xacro:property name="calf_ixx" value="0.0028925"/>
-	<xacro:property name="calf_ixy" value="-0.00000012574"/>
-	<xacro:property name="calf_ixz" value="0.00013889"/>
-	<xacro:property name="calf_iyy" value="0.0029343"/>
-	<xacro:property name="calf_iyz" value="0.0000004083"/>
-	<xacro:property name="calf_izz" value="0.000082284"/>
-	<xacro:property name="calf_rotor_mass" value="0.089"/>
+	<xacro:property name="calf_ixx" value="0.003018669"/>
+	<xacro:property name="calf_ixy" value="-0.000000131225"/>
+	<xacro:property name="calf_ixz" value="0.000144948"/>
+	<xacro:property name="calf_iyy" value="0.003062293"/>
+	<xacro:property name="calf_iyz" value="0.000000426110"/>
+	<xacro:property name="calf_izz" value="0.0000858732"/>
+	<xacro:property name="calf_rotor_mass" value="0.092882"/>
 	<xacro:property name="calf_rotor_com_x" value="0.0"/>
 	<xacro:property name="calf_rotor_com_y" value="0.0"/>
 	<xacro:property name="calf_rotor_com_z" value="0.0"/>
-	<xacro:property name="calf_rotor_ixx" value="0.000059647"/>
+	<xacro:property name="calf_rotor_ixx" value="0.000062249"/>
 	<xacro:property name="calf_rotor_ixy" value="0.0"/>
 	<xacro:property name="calf_rotor_ixz" value="0.0"/>
-	<xacro:property name="calf_rotor_iyy" value="0.000111842"/>
+	<xacro:property name="calf_rotor_iyy" value="0.000116720"/>
 	<xacro:property name="calf_rotor_iyz" value="0.0"/>
-	<xacro:property name="calf_rotor_izz" value="0.000059647"/>
+	<xacro:property name="calf_rotor_izz" value="0.000062249"/>
 	<!-- foot -->
-	<xacro:property name="foot_mass" value="0.06"/>
+	<xacro:property name="foot_mass" value="0.062617"/>
 </robot>
