Commit message: para_ident10.19

File: src/quadruped_ros2_control-humble/descriptions/sysu219/sysu219_description/xacro/robot.xacro (robot description, xacro)
@@ -47,5 +47,5 @@
 	<link name="trunk">
 		<visual>
-			<origin rpy="0 0 0" xyz="0 0 0"/>
+			<origin rpy="${PI} 0 0" xyz="0 0 0"/>
 			<geometry>
 				<mesh filename="file://$(find sysu219_description)/meshes/trunk.dae" scale="0.001 0.001 0.001"/>
